File: servo motor tester/servo motor tester.kicad_pcb (KiCad board)
At the start: 2 copper layers, 44.8 x 27.6 mm, 10 parts, among them J1 Conn_01x02_Pin, J2 Conn_01x03_Pin, U1 NE555P

Commit message: update project
Parts:
- C1: footprint Capacitor_THT:CP_Radial_D4.0mm_P1.50mm -> Capacitor_THT:C_Disc_D3.8mm_W2.6mm_P2.50mm
- J1: footprint Connector_PinHeader_1.00mm:PinHeader_1x02_P1.00mm_Horizontal -> Connector_PinHeader_2.54mm:PinHeader_1x02_P2.54mm_Horizontal
- J2: footprint Connector_PinHeader_1.00mm:PinHeader_1x03_P1.00mm_Horizontal -> Connector_PinHeader_2.54mm:PinHeader_1x03_P2.54mm_Horizontal
- RV1: footprint Potentiometer_THT:Potentiometer_ACP_CA6-H2,5_Horizontal -> Potentiometer_THT:Potentiometer_Alps_RK163_Single_Horizontal
- moved D1 50.9 mm to (111.5, 96.0), turned to 0 degrees
- moved R2 40.4 mm to (111.5, 74.9), turned to -90 degrees
- moved R1 36.6 mm to (121.6, 101.0), turned to 180 degrees
- moved RV1 31.9 mm to (129.0, 77.5)
- moved C1 31.5 mm to (136.0, 83.0), turned to 90 degrees
- moved U1 28.6 mm to (119.2, 89.2), turned to 0 degrees
- moved J2 27.8 mm to (136.0, 90.4)
- moved J1 21.6 mm to (113.5, 91.5)
- moved D2 18.5 mm to (131.5, 97.3), turned to 90 degrees
- moved R3 16.0 mm to (136.6, 102.0), turned to 180 degrees
Routing:
- net Net-(D2-K): track 83.2 -> 43.0 mm
- net GND: track 31.3 -> 0.00 mm
- net Net-(J1-Pin_1): track 41.6 -> 70.9 mm
- net Net-(R3-Pad1): track 10.7 -> 35.3 mm
- net Net-(D2-A): track 40.3 -> 34.4 mm
- net Net-(D1-A): track 4.47 -> 8.68 mm
- net Net-(J2-Pin_3): track 22.2 -> 21.7 mm
Other:
- board size 44.8 x 27.6 mm -> 32.5 x 32 mm
- board text added: "servo tester"
