File: USB to UART/USB to UART.kicad_sch (KiCad schematic)
At the start: 19 parts, among them J1 USB_C_Receptacle_USB2.0_16P, J2 Conn_01x05_Pin, U1 CP2102N-Axx-xQFN28

Commit message: screenshot added
Changed lines of the file:
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@@
 			(font
 				(size 3 3)
-				(thickness 0.254)
+				(thickness 0.6)
 				(bold yes)
 			)
