File: ncv_detector/ncv_detector.kicad_sch (KiCad schematic)
At the start: 10 parts, among them Q1 2N3904, Q2 2N3904, Q3 2N3904

Commit message: screenshot added
Parts:
- BT1: footprint Battery:BatteryHolder_Keystone_1042_1x18650 -> Battery:BatteryHolder_Bulgin_BX0034_1xAAA
Other:
- note added: "NCV DETECTOR"
- company: (none) -> Av_Designs
- title: (none) -> NCV DETECTOR
- moved on the sheet: AE1, BT1, BZ1, D1, Q1, Q2, Q3, R1, R2, R3
